Commit message: Added launch file to enable gazebo and rviz

File: ros_package/my_navigation_impl/urdf/my_navigation_impl.urdf (robot description, URDF)
Before this commit: robot my_navigation_impl, 6 links, 5 joints
Links:
- removed link hokuyo_link
- added link lidar_link, mass 1e-5; collision box size=0.1 0.1 0.1; visual box size=0.05 0.05 0.01
Joints:
- joint hokuyo_joint: child hokuyo_link -> lidar_link; origin xyz=0 0 0.9 rpy=0 0 0 -> xyz=0 0 0.1 rpy=0 0 0
