Commit message: Added custom world and spawned robot in new world

File: ros_package/my_navigation_impl/urdf/cpy_my_navigation_impl.urdf (robot description, URDF)
Before this commit: robot my_navigation_impl, 5 links, 4 joints
Links:
- added link lidar_link, mass 1e-5; collision box size=0.1 0.1 0.1; visual box size=0.05 0.05 0.01
Joints:
- added joint hokuyo_joint: type fixed, parent base_link, child lidar_link, origin xyz=0 0 0.1 rpy=0 0 0, axis 0 1 0
