Commit message: Fixed the issue with joint configuration and laser scan topic

File: ros_package/ddrive_navigation_impl/urdf/ddrive_navigation_impl.urdf (robot description, URDF)
Before this commit: robot ddrive_navigation_impl, 3 links, 2 joints
Joints:
- joint right_joint: axis 0 0 1 -> 0 0 -1

File: ros_package/ddrive_navigation_impl/urdf/ddrive_navigation_impl_integration.urdf.xacro (robot description, xacro)
@@ -32,7 +32,7 @@
 		<sensor name="laser" type="ray">
 			<!-- Add in your sensor characteristics -->
-			<pose> 0 0 0.06 0 0 0 </pose>
+			<pose> 0.02 0 0.06 0 0 0 </pose>
 			<visualise>true</visualise>
-			<update_rate>20</update_rate>
+			<update_rate>30</update_rate>
 			<ray>
 				<scan>
@@ -57,5 +57,5 @@
 			<plugin name="gazebo_ros_head_hokuyo_controller" filename="libgazebo_ros_laser.so">
 				<!-- Use topic name as /my_robot/scan -->
-					<topicName>/laser/scan</topicName>
+					<topicName>/scan</topicName>
 					<frameName>base_laser</frameName>
 			</plugin>
